Commit message: Copied a ROS example file (single_link something) to get the basics of a shoulder joint working. Having trouble with the collision though so it's bouncing all over the place

File: gaffa_common/gaffa_description/robots/gaffa.urdf.xacro (robot description, xacro)
@@ -1,21 +1,152 @@
 <?xml version="1.0"?>
+<robot name="pr2"
+       xmlns:xi="http://www.w3.org/2001/XInclude"
+       xmlns:gazebo="http://playerstage.sourceforge.net/gazebo/xmlschema/#gz"
+       xmlns:model="http://playerstage.sourceforge.net/gazebo/xmlschema/#model"
+       xmlns:sensor="http://playerstage.sourceforge.net/gazebo/xmlschema/#sensor"
+       xmlns:body="http://playerstage.sourceforge.net/gazebo/xmlschema/#body"
+       xmlns:geom="http://playerstage.sourceforge.net/gazebo/xmlschema/#geom"
+       xmlns:joint="http://playerstage.sourceforge.net/gazebo/xmlschema/#joint"
+       xmlns:interface="http://playerstage.sourceforge.net/gazebo/xmlschema/#interface"
+       xmlns:rendering="http://playerstage.sourceforge.net/gazebo/xmlschema/#rendering"
+       xmlns:renderable="http://playerstage.sourceforge.net/gazebo/xmlschema/#renderable"
+       xmlns:controller="http://playerstage.sourceforge.net/gazebo/xmlschema/#controller"
+       xmlns:physics="http://playerstage.sourceforge.net/gazebo/xmlschema/#physics">
+  <joint name="base_block_joint" type="fixed">
+    <parent link="world" />
+    <origin xyz="0 0 0" rpy="0 0 0" />
+    <child link="base_block" />
+  </joint>
+  <property name="M_PI" value="3.1415926535897931" />
+  <link name="base_block">
+    <inertial>
+      <mass value="1000" />
+      <origin xyz="0 0 0" />
+      <inertia ixx="100"  ixy="0"  ixz="0" iyy="100" iyz="0" izz="100" />
+    </inertial>
+    <visual>
+      <origin xyz="0 0 0" rpy="0 0 0" />
+      <geometry name="base_block_visual_geom">
+        <box size="0.3 0.14 0.01" />
+      </geometry>
+    </visual>
+    <collision>
+      <origin xyz="0 0 0" rpy="0.0 0.0 0.0" />
+      <geometry name="base_block_collision_geom">
+        <box size="0.3 0.14 0.01" />
+      </geometry>
+    </collision>
+  </link>
+  <gazebo reference="base_block">
+    <material>Gazebo/GrassFloor</material>
+    <turnGravityOff>true</turnGravityOff>
+    <selfCollide>false</selfCollide>
+  </gazebo>
+  <joint name="base_rotate_joint" type="revolute" >
+    <axis xyz="0 0 1" />
+    <limit upper="${M_PI/2}" lower="${-M_PI/2}" effort="100" velocity="5" />
+    <parent link="base_block" />
+    <origin xyz="0 0 0.061" rpy="0 0 0" />
+    <child link="base_rotate_link" />
+  </joint>
+  <link name="base_rotate_link">
+    <inertial >
+      <mass value="10" />
+      <origin xyz="0.4 0 0" />
+      <inertia  ixx="0.1" ixy="0.0"  ixz="0.0"  iyy="0.1"  iyz="0.0"  izz="0.018" />
+    </inertial>
+    <visual >
+      <origin xyz="0.0 0 -0.025" rpy="0 0 0" />
+      <geometry name="base_rotate_mesh_file">
+        <cylinder radius="0.06" length="0.05" />
+      </geometry>
+    </visual>
+    <collision >
+      <origin xyz="0.0 0 -0.025" rpy="0 0 0" />
+      <geometry name="base_rotate_collision_geom">
+        <cylinder radius="0.06" length="0.05" />
+      </geometry>
+    </collision>
+  </link>
+  <gazebo reference="base_rotate_link">
+    <material>Gazebo/Red</material>
+    <turnGravityOff>true</turnGravityOff>
+    <selfCollide>false</selfCollide>
+  </gazebo>
+  <joint name="shoulder_rotate_joint" type="revolute" >
+    <axis xyz="0 1 0" />
+    <limit upper="0" lower="${-3*M_PI/4}" effort="100" velocity="5" />
+    <parent link="base_rotate_link" />
+    <origin xyz="0 0 0.025" rpy="0 0 0" />
+    <child link="upper_arm_link" />
+  </joint>
+  <link name="upper_arm_link">
+    <inertial >
+      <mass value="10" />
+      <origin xyz="0.08 0 0" />
+      <inertia  ixx="0.1" ixy="0.0"  ixz="0.0"  iyy="0.1"  iyz="0.0"  izz="0.1" />
+    </inertial>
+    <visual >
+      <origin xyz="0.08 0 0.0" rpy="0 0 0" />
+      <geometry name="upper_arm_mesh_file">
+        <box size="0.2 0.05 0.05" />
+      </geometry>
+    </visual>
+    <collision >
+      <origin xyz="0.08 0 0.0" rpy="0 0 0" />
+      <geometry name="upper_arm_collision_geom">
+        <box size="0.2 0.05 0.05" />
+      </geometry>
+    </collision>
+  </link>
+  <gazebo reference="upper_arm_link">
+    <material>Gazebo/Blue</material>
+    <turnGravityOff>true</turnGravityOff>
+    <selfCollide>false</selfCollide>
+  </gazebo>
+  <gazebo>
+      <controller:gazebo_ros_time name="gazebo_ros_time" plugin="libgazebo_ros_time.so">
+        <alwaysOn>true</alwaysOn>
+        <updateRate>1000.0</updateRate>
+        <interface:audio name="dummy_gazebo_ros_time_iface_should_not_be_here"/>
+      </controller:gazebo_ros_time>
+      <!-- PR2_ACTARRAY -->
+<!--      <controller:gazebo_ros_controller_manager name="gazebo_ros_controller_manager" plugin="libgazebo_ros_controller_manager.so">
+        <alwaysOn>true</alwaysOn>
+        <updateRate>1000.0</updateRate>
+        <interface:audio name="gazebo_ros_controller_manager_dummy_iface" />
+      </controller:gazebo_ros_controller_manager>-->
+      <!-- gazebo_ros_p3d for position groundtruth -->
+<!--      <controller:gazebo_ros_p3d name="p3d_link1_controller" plugin="libgazebo_ros_p3d.so">
+          <alwaysOn>true</alwaysOn>
+          <updateRate>1000.0</updateRate>
+          <bodyName>link1</bodyName>
+          <topicName>link1_pose</topicName>
+          <frameName>map</frameName>
+          <interface:position name="p3d_link1_position"/>
+      </controller:gazebo_ros_p3d>-->
+  </gazebo>
+  <!-- mechanism controls -->
+<!--   <include filename="./single_link.transmission.xacro" /> -->
+</robot>
+<!--<?xml version="1.0"?>
 <robot xmlns:sensor="http://playerstage.sourceforge.net/gazebo/xmlschema/#sensor"
        xmlns:controller="http://playerstage.sourceforge.net/gazebo/xmlschema/#controller"
        xmlns:interface="http://playerstage.sourceforge.net/gazebo/xmlschema/#interface"
        xmlns:xacro="http://playerstage.sourceforge.net/gazebo/xmlschema/#interface"
-       name="pr2" >
+       name="pr2" >-->
   <!-- The following included files set up definitions of parts of the robot body -->
   <!-- misc common stuff? -->
-  <include filename="$(find gaffa_description)/urdf/common.xacro" />
-  <!-- Maplin Arm -->
-  <include filename="$(find gaffa_description)/urdf/maplin_upper_arm/maplin_upper_arm.urdf.xacro" />
-  <!-- Maplin gripper -->
+  <!--<include filename="$(find gaffa_description)/urdf/common.xacro" />
+  --><!-- Maplin Arm -->
+ <!-- <include filename="$(find gaffa_description)/urdf/maplin_upper_arm/maplin_upper_arm.urdf.xacro" />
+  --><!-- Maplin gripper -->
   <!--<include filename="$(find gaffa_description)/urdf/maplin_gripper.urdf.xacro" />-->
   <!-- Gaffa base -->
-  <include filename="$(find gaffa_description)/urdf/base/base.urdf.xacro" />
+<!--   <include filename="$(find gaffa_description)/urdf/base/base.urdf.xacro" /> -->
   <!-- generic simulator_gazebo plugins for starting mechanism control, ros time, ros battery -->
   <!--<include filename="$(find pr2_description)/gazebo/gazebo.urdf.xacro" />-->
   <!-- materials for visualization -->
-  <include filename="$(find pr2_description)/urdf/materials.urdf.xacro" />
+<!--   <include filename="$(find pr2_description)/urdf/materials.urdf.xacro" /> -->
   <!-- Now we can start using the macros included above to define the actual PR2 -->
   <!-- The first use of a macro.  This one was defined in base.urdf.xacro above.
@@ -26,5 +157,5 @@
        the origin block defines where the component is w.r.t its parent (in this case the parent
        is the world frame). For more, see http://www.ros.org/wiki/xacro -->
-  <xacro:gaffa_base name="base"/>
-  <xacro:maplin_upper_arm side="r" reflect="-1" parent="base_link"/>
-</robot>
+<!--   <xacro:gaffa_base name="base"/> -->
+<!--   <xacro:maplin_upper_arm side="r" reflect="-1" parent="base_link"/> -->
+<!-- </robot> -->
