Commit message: Got the simulated version of the SSC32 server working with the simulator and the Gaffa_Teleop program. Controlling the simulated arm with forces is turning out to be a bit tricky however so it may be better to fall back to a simpler simulation where the angles are set directly

File: gaffa_common/gaffa_description/robots/gaffa.urdf.xacro (robot description, xacro)
@@ -19,5 +19,5 @@
   </joint>-->
   <property name="M_PI" value="3.1415926535897931" />
-  <property name="BASE_MASS" value="10" />
+  <property name="BASE_MASS" value="100" />
   <property name="BASE_LENGTH" value="0.3" />
   <property name="BASE_WIDTH" value="0.15" />
@@ -29,5 +29,5 @@
   <property name="UPPER_ARM_MASS" value="0.1" />
   <property name="UPPER_ARM_LENGTH" value="0.154" />
-  <property name="UPPER_ARM_WIDTH" value="0.053" />
+  <property name="UPPER_ARM_WIDTH" value="0.052" />
   <property name="UPPER_ARM_HEIGHT" value="0.0244" />
   <!-- Mass includes both elbow and wrist servos -->
@@ -39,5 +39,5 @@
   <property name="WRIST_MASS" value="0.065" />
   <property name="WRIST_LENGTH" value="0.0346" />
-  <property name="WRIST_WIDTH" value="0.053" />
+  <property name="WRIST_WIDTH" value="0.052" />
   <property name="WRIST_HEIGHT" value="0.0244" />
   <!-- Mass includes gripper 'grip' servo -->
@@ -118,5 +118,5 @@
   <joint name="shoulder_rotate_joint" type="revolute" >
     <axis xyz="0 0 1" />
-    <limit upper="${M_PI/2}" lower="0" effort="100" velocity="5" />
+    <limit upper="${3*M_PI/4}" lower="0" effort="100" velocity="5" />
     <parent link="base_rotate_link" />
     <origin xyz="0 0 ${SHOULDER_HEIGHT - BASE_ROTATE_HEIGHT/2}" rpy="${M_PI/2} 0 0" />
@@ -190,7 +190,7 @@
   <joint name="wrist_rotate_joint" type="revolute" >
     <axis xyz="0 0 1" />
-    <limit upper="${M_PI/2}" lower="${-M_PI/2}" effort="100" velocity="5" />
+    <limit upper="${M_PI}" lower="${0}" effort="100" velocity="5" />
     <parent link="fore_arm_link" />
-    <origin xyz="${FORE_ARM_LENGTH} 0 0.0" rpy="0 0 0" />
+    <origin xyz="${FORE_ARM_LENGTH} 0 0.0" rpy="0 0 ${-M_PI/2}" />
     <child link="wrist_link" />
   </joint>

Commit message: First pass changes to add a camera to the robot both in the simulator and the real world

File: gaffa_common/gaffa_description/robots/gaffa.urdf.xacro (robot description, xacro)
@@ -331,4 +331,40 @@
     <selfCollide>true</selfCollide>
   </gazebo>
+  <!-- Gripper camera -->
+  <joint name="gripper_camera_joint" type="fixed" >
+    <axis xyz="1 0 0" />
+    <limit upper="0" lower="0" effort="100" velocity="5" />
+    <parent link="gripper_base_link" />
+    <origin xyz="0 0 ${GRIPPER_BASE_LENGTH + 0.02}" rpy="0 ${-M_PI/2} ${-M_PI/2}" />
+    <child link="gripper_camera_link" />
+  </joint>
+  <link name="gripper_camera_link">
+    <inertial >
+      <mass value="0.0001" />
+      <origin xyz="${GRIPPER_FINGER_LENGTH/2} 0 0" />
+      <inertia ixx="${GRIPPER_FINGER_MASS*(GRIPPER_FINGER_LENGTH*GRIPPER_FINGER_LENGTH + GRIPPER_FINGER_HEIGHT*GRIPPER_FINGER_HEIGHT)/12.0}"
+               ixy="0" ixz="0"
+               iyy="${GRIPPER_FINGER_MASS*(GRIPPER_FINGER_LENGTH*GRIPPER_FINGER_LENGTH + GRIPPER_FINGER_WIDTH*GRIPPER_FINGER_WIDTH)/12.0}"
+               iyz="0"
+               izz="${GRIPPER_FINGER_MASS*(GRIPPER_FINGER_WIDTH*GRIPPER_FINGER_WIDTH + GRIPPER_FINGER_HEIGHT*GRIPPER_FINGER_HEIGHT)/12.0}" />
+    </inertial>
+    <visual >
+      <origin xyz="0 0 ${GRIPPER_FINGER_LENGTH/2}" rpy="0 0 0" />
+      <geometry name="gripper_finger_visual_geom">
+        <box size="${GRIPPER_FINGER_WIDTH} ${GRIPPER_FINGER_HEIGHT} ${GRIPPER_FINGER_LENGTH}" />
+      </geometry>
+    </visual>
+    <collision >
+      <origin xyz="0 0 ${GRIPPER_FINGER_LENGTH/2}" rpy="0 0 0" />
+      <geometry name="gripper_finger_collision_geom">
+        <box size="${GRIPPER_FINGER_WIDTH} ${GRIPPER_FINGER_HEIGHT} ${GRIPPER_FINGER_LENGTH}" />
+      </geometry>
+    </collision>
+  </link>
+  <gazebo reference="gripper_camera_link">
+    <material>Gazebo/Blue</material>
+    <turnGravityOff>false</turnGravityOff>
+    <selfCollide>false</selfCollide>
+  </gazebo>
   <gazebo>
       <controller:gazebo_ros_time name="gazebo_ros_time" plugin="libgazebo_ros_time.so">
@@ -353,4 +389,25 @@
       </controller:gazebo_ros_p3d>-->
   </gazebo>
+  <!-- Camera -->
+  <gazebo reference="gripper_camera_link">
+      <sensor:camera name="gripper_camera_sensor">
+        <imageSize>320 240</imageSize>
+        <imageFormat>L8</imageFormat>
+        <hfov>45</hfov>
+        <nearClip>0.01</nearClip>
+        <farClip>100</farClip>
+        <updateRate>20.0</updateRate>
+        <controller:gazebo_ros_camera name="gripper_camera_controller" plugin="libgazebo_ros_camera.so">
+          <alwaysOn>true</alwaysOn>
+          <updateRate>20.0</updateRate>
+          <imageTopicName>gripper_cam/image</imageTopicName>
+          <cameraInfoTopicName>gripper_cam/info</cameraInfoTopicName>
+          <frameName>gripper_camera</frameName>
+          <interface:camera name="gripper_camera_iface" />
+        </controller:gazebo_ros_camera>
+      </sensor:camera>
+      <!--<turnGravityOff>true</turnGravityOff>
+      <material>PR2/Blue</material>-->
+    </gazebo>
   <!-- mechanism controls -->
   <transmission type="pr2_mechanism_model/SimpleTransmission" name="base_rotate_trans">
